File: icom/icom-ci-v.kicad_pcb (KiCad board)
At the start: 2 copper layers, 33.8 x 28.4 mm, 10 parts, among them J1 Conn_01x06_Male, J2 Conn_01x02_Female, J3 Conn_01x02_Female, Q1 BSS138, U1 74LVC2G125, X1 Würth_615008138221

Commit message: PCB: cleanups
Parts:
- moved C1 8.58 mm to (137.4, 83.1), turned to 0 degrees
- moved R1 1.00 mm to (133.1, 87.0)
- moved U1 1.00 mm to (137.2, 85.8)
- turned R3 to 180 degrees
Routing:
- net +3.3V: track 25.4 -> 22.5 mm
- net /TX: track 7.54 -> 9.80 mm
- net /PTT: track 16.9 -> 14.7 mm
- net /CIV-RADIO-CLONE: track 5.05 -> 6.62 mm
- net Net-(Q1-Pad1): track 2.10 -> 3.46 mm
- net /RX: track 7.02 -> 7.54 mm
- net GND: vias 1 -> 5

Commit message: Moved J1 and J2 to give clearance for the plug against the RJ45 connector
Parts:
- moved J2 4.22 mm to (140.0, 63.5)
- moved J3 4.22 mm to (129.3, 63.5)
Routing:
- net /PTT: track 14.7 -> 18.9 mm
- net /CIV-RADIO-MICE: track 16.7 -> 20.9 mm
- net /CIV-RADIO-MIC: track 13.6 -> 17.9 mm
Other:
- board size 33.8 x 28.4 mm -> 33.8 x 32.8 mm
Changed lines of the file:
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@@
   (net 15 "/CIV-RADIO-MICE")
   (footprint "Connector_Phoenix_MC:PhoenixContact_MCV_1,5_2-G-3.5_1x02_P3.50mm_Vertical" (layer "F.Cu")
-    (at 129.3315 67.6985)
+    (at 129.3114 63.4746)
     (descr "Generic Phoenix Contact connector footprint for: MCV_1,5/2-G-3.5; number of pins: 02; pin pitch: 3.50mm; Vertical || order number: 1843606 8A 160V")
     (tags "phoenix_contact connector MCV_01x02_G_3.5mm")
@@
   )
   (footprint "Connector_Phoenix_MC:PhoenixContact_MCV_1,5_2-G-3.5_1x02_P3.50mm_Vertical" (layer "F.Cu")
-    (at 139.9995 67.6985)
+    (at 139.9794 63.4746)
     (descr "Generic Phoenix Contact connector footprint for: MCV_1,5/2-G-3.5; number of pins: 02; pin pitch: 3.50mm; Vertical || order number: 1843606 8A 160V")
     (tags "phoenix_contact connector MCV_01x02_G_3.5mm")
@@
     )
   )
-  (gr_rect (start 125.476 62.484) (end 159.258 90.932) (layer "Edge.Cuts") (width 0.1) (fill none))
-  (gr_text "iCOM CI-V\nTester v1.0" (at 153.416 65.024) (layer "F.SilkS")
-    (effects (font (size 1 1) (thickness 0.15)))
+  (gr_rect (start 125.476 58.166) (end 159.258 90.932) (layer "Edge.Cuts") (width 0.1) (fill none))
+  (gr_text "iCOM CI-V Tester\nv1.0" (at 157.48 59.944 45) (layer "F.SilkS")
+    (effects (font (size 1 1) (thickness 0.15)) (justify right))
   )
   (segment (start 136.2964 86.594) (end 136.2964 86.1876) (width 0.25) (layer "F.Cu") (net 1))
@@
   (segment (start 141.044 80.264) (end 142.695 81.915) (width 0.25) (layer "F.Cu") (net 8))
   (segment (start 139.1135 80.264) (end 141.044 80.264) (width 0.25) (layer "F.Cu") (net 8))
-  (segment (start 135.128 73.584) (end 132.8315 71.2875) (width 0.25) (layer "F.Cu") (net 9))
   (segment (start 137.2385 77.216) (end 135.86 77.216) (width 0.25) (layer "F.Cu") (net 9))
+  (segment (start 132.8114 67.0254) (end 132.8114 63.4746) (width 0.25) (layer "F.Cu") (net 9))
   (segment (start 135.128 79.439) (end 135.128 77.948) (width 0.25) (layer "F.Cu") (net 9))
-  (segment (start 135.128 76.484) (end 135.128 76.2) (width 0.25) (layer "F.Cu") (net 9))
-  (segment (start 132.8315 71.2875) (end 132.8315 67.6985) (width 0.25) (layer "F.Cu") (net 9))
+  (segment (start 135.128 77.948) (end 135.86 77.216) (width 0.25) (layer "F.Cu") (net 9))
+  (segment (start 135.128 76.484) (end 135.128 69.342) (width 0.25) (layer "F.Cu") (net 9))
+  (segment (start 135.128 69.342) (end 132.8114 67.0254) (width 0.25) (layer "F.Cu") (net 9))
   (segment (start 135.86 77.216) (end 135.128 76.484) (width 0.25) (layer "F.Cu") (net 9))
-  (segment (start 135.128 76.2) (end 135.128 73.584) (width 0.25) (layer "F.Cu") (net 9))
-  (segment (start 135.128 77.948) (end 135.86 77.216) (width 0.25) (layer "F.Cu") (net 9))
   (segment (start 139.31 85.507) (end 141.643 85.507) (width 0.25) (layer "F.Cu") (net 10))
   (segment (start 141.643 85.507) (end 142.695 84.455) (width 0.25) (layer "F.Cu") (net 10))
@@
   (segment (start 140.137 86.157) (end 140.462 85.832) (width 0.25) (layer "F.Cu") (net 10))
   (segment (start 142.639 84.511) (end 142.695 84.455) (width 0.25) (layer "F.Cu") (net 10))
-  (segment (start 143.4995 67.6985) (end 143.4995 70.0185) (width 0.25) (layer "F.Cu") (net 11))
-  (segment (start 143.4995 70.0185) (end 140.716 72.802) (width 0.25) (layer "F.Cu") (net 11))
-  (segment (start 140.716 72.802) (end 140.716 77.396) (width 0.25) (layer "F.Cu") (net 11))
+  (segment (start 143.4794 63.4746) (end 143.4794 67.0866) (width 0.25) (layer "F.Cu") (net 11))
+  (segment (start 143.4794 67.0866) (end 140.716 69.85) (width 0.25) (layer "F.Cu") (net 11))
   (segment (start 140.716 77.396) (end 142.695 79.375) (width 0.25) (layer "F.Cu") (net 11))
-  (segment (start 139.9995 67.6985) (end 139.9995 78.134726) (width 0.25) (layer "F.Cu") (net 15))
-  (segment (start 142.509774 80.645) (end 145.235 80.645) (width 0.25) (layer "F.Cu") (net 15))
-  (segment (start 139.9995 78.134726) (end 142.509774 80.645) (width 0.25) (layer "F.Cu") (net 15))
+  (segment (start 140.716 69.85) (end 140.716 77.396) (width 0.25) (layer "F.Cu") (net 11))
+  (segment (start 139.9995 78.134726) (end 139.9995 63.4947) (width 0.25) (layer "F.Cu") (net 15))
+  (segment (start 139.9995 63.4947) (end 139.9794 63.4746) (width 0.25) (layer "F.Cu") (net 15))
+  (segment (start 142.509774 80.645) (end 139.9995 78.134726) (width 0.25) (layer "F.Cu") (net 15))
+  (segment (start 145.235 80.645) (end 142.509774 80.645) (width 0.25) (layer "F.Cu") (net 15))
   (zone (net 1) (net_name "GND") (layers F&B.Cu) (hatch edge 0.508)
     (connect_pads (clearance 0.508))
@@
         (xy 158.75 90.424)
         (xy 125.984 90.424)
-        (xy 125.984 62.992)
-        (xy 158.75 62.992)
+        (xy 125.984 58.674)
+        (xy 158.75 58.674)
       )
     )
